File: hardware/rev_a/rumblecation+ble.sch (EAGLE design)
At the start: 76 parts, among them J1 FCI_CORTEX_SWD_CONNECTOR, J2 JST_S2B-PH-SM4-TB_CONNECTOR, J3 MINI_USB_B, J6 TC2030-JLINK-NL, M1 PRECISION_MICRODRIVES_C100-10, M2 PRECISION_MICRODRIVES_310-113, U1 ATSAMD4S2BA-AU, U2 SILABS_CP2102, U3 TLV73333PDBVT, U4 TI_DRV2603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

Commit message: fixed silab usb-uart, added fsync and int to accell, updated schematic prettiness, fixed regout on accel
Parts:
- added C32: 4.7uF, rumbleaction_parts_lib:C-USC0402
- added C33: 100nF, rumbleaction_parts_lib:C-USC0402
- U1: value ATSAMD4S2BA-AU -> ATSAM4S2BA-AU
Connections:
- net D+ renamed USB_D_P
- net D- renamed USB_D_N
- net N$4 renamed USB_LED
- new net MPU_FSYNC: U1.PA26/PGMD14, U6.FSYNC, U7.FSYNC
- new net MPU_INT: U1.PA25/PGMD13, U6.INT, U7.INT
- net +3V3: now also C32.1, C33.1, U2.REGIN
- net GND: now also C32.2, C33.2
- net VBUS: no longer U2.REGIN
Other:
- moved on the sheet: C1, C10, C11, C12, C13, C14, C15, C16, C18, C19, C20, C22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

Commit message: Added a power selector header, fixed some routing errors
Parts:
- added JP1: (no value), SparkFun-Connectors:M03PTH
Connections:
- new net N$4: JP1.2, U3.EN, U3.VIN
- net N$7: now also JP1.1; no longer U3.EN, U3.VIN
- net VBUS: now also JP1.3
Changed lines of the file:
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@@
 <part name="C33" library="rumbleaction_parts_lib" deviceset="C-US" device="C0402" value="100nF"/>
 <part name="GND56" library="supply1" deviceset="GND" device=""/>
+<part name="JP1" library="SparkFun-Connectors" deviceset="M03" device="PTH"/>
 </parts>
 <sheets>
@@
 <text x="109.22" y="177.8" size="1.778" layer="91">VDDIO</text>
 <text x="175.26" y="177.8" size="1.778" layer="91">VDDCORE</text>
-<text x="33.02" y="119.38" size="1.778" layer="91">3.3V Power</text>
+<text x="38.1" y="116.84" size="1.778" layer="91">3.3V Power</text>
 <text x="38.1" y="167.64" size="1.778" layer="91">SWD connector</text>
 <text x="132.08" y="132.08" size="1.778" layer="91">Main MCU</text>
@@
 <instance part="GND54" gate="1" x="48.26" y="22.86" rot="R90"/>
 <instance part="GND55" gate="1" x="48.26" y="10.16" rot="R90"/>
+<instance part="JP1" gate="G$1" x="22.86" y="134.62" rot="R270"/>
 </instances>
 <busses>
@@
 </segment>
 </net>
-<net name="N$7" class="0">
-<segment>
-<pinref part="J2" gate="G$1" pin="VCC"/>
-<pinref part="U3" gate="G$1" pin="VIN"/>
-<wire x1="17.78" y1="111.76" x2="25.4" y2="111.76" width="0.1524" layer="91"/>
-<pinref part="U3" gate="G$1" pin="EN"/>
-<wire x1="25.4" y1="111.76" x2="27.94" y2="111.76" width="0.1524" layer="91"/>
-<wire x1="27.94" y1="106.68" x2="25.4" y2="106.68" width="0.1524" layer="91"/>
-<wire x1="25.4" y1="106.68" x2="25.4" y2="111.76" width="0.1524" layer="91"/>
-<junction x="25.4" y="111.76"/>
-</segment>
-</net>
 <net name="LRA_PWM" class="0">
 <segment>
@@
 </segment>
 </net>
+<net name="N$4" class="0">
+<segment>
+<pinref part="JP1" gate="G$1" pin="2"/>
+<wire x1="22.86" y1="127" x2="22.86" y2="111.76" width="0.1524" layer="91"/>
+<pinref part="U3" gate="G$1" pin="VIN"/>
+<wire x1="22.86" y1="111.76" x2="25.4" y2="111.76" width="0.1524" layer="91"/>
+<wire x1="25.4" y1="111.76" x2="27.94" y2="111.76" width="0.1524" layer="91"/>
+<wire x1="25.4" y1="111.76" x2="25.4" y2="106.68" width="0.1524" layer="91"/>
+<pinref part="U3" gate="G$1" pin="EN"/>
+<wire x1="25.4" y1="106.68" x2="27.94" y2="106.68" width="0.1524" layer="91"/>
+</segment>
+</net>
+<net name="N$7" class="0">
+<segment>
+<pinref part="J2" gate="G$1" pin="VCC"/>
+<pinref part="JP1" gate="G$1" pin="1"/>
+<wire x1="17.78" y1="111.76" x2="20.32" y2="111.76" width="0.1524" layer="91"/>
+<wire x1="20.32" y1="111.76" x2="20.32" y2="127" width="0.1524" layer="91"/>
+</segment>
+</net>
+<net name="VBUS" class="0">
+<segment>
+<pinref part="JP1" gate="G$1" pin="3"/>
+<wire x1="25.4" y1="127" x2="25.4" y2="119.38" width="0.1524" layer="91"/>
+<wire x1="25.4" y1="119.38" x2="33.02" y2="119.38" width="0.1524" layer="91"/>
+<wire x1="33.02" y1="119.38" x2="33.02" y2="124.46" width="0.1524" layer="91"/>
+<label x="33.02" y="124.46" size="1.778" layer="95" rot="R90" xref="yes"/>
+</segment>
+</net>

Commit message: Final board revision - being sent for production
Changed lines of the file:
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@@
 <pinref part="U3" gate="G$1" pin="EN"/>
 <wire x1="25.4" y1="106.68" x2="27.94" y2="106.68" width="0.1524" layer="91"/>
+<junction x="25.4" y="111.76"/>
 </segment>
 </net>
@@
 <pinref part="C33" gate="G$1" pin="1"/>
 <wire x1="147.32" y1="101.6" x2="147.32" y2="106.68" width="0.1524" layer="91"/>
-</segment>
-</net>
+<junction x="147.32" y="106.68"/>
+<junction x="157.48" y="106.68"/>
+</segment>
+</net>
